File: plytkamh/plytkamh.kicad_pcb (KiCad board)
At the start: 2 copper layers, 70 x 50 mm, 57 parts, among them J1 USB_C_Receptacle_USB2.0_16P, J2 BOOT0, J3 Conn_01x06, J4 COMM, J5 ANALOG_GPIO, Q1 TEMT6000X01, SW1 RESET, SW2 USER, U1 USBLC6-2SC6, U2 LDL1117S33R, U3 STM32F446RETx, U4 BME280, Y1 12MHz

Commit message: Before board resize
Parts:
- moved C15 163.6 mm to (165.2, 140.0), turned to 180 degrees
- moved R5 157.5 mm to (167.1, 132.9), turned to 180 degrees
- moved C16 157.2 mm to (161.6, 136.8), turned to -90 degrees
- moved R6 153.8 mm to (163.4, 134.2), turned to 180 degrees
- moved C13 151.7 mm to (152.7, 131.2)
- moved C14 150.8 mm to (157.1, 127.2), turned to -90 degrees
- moved R7 147.0 mm to (161.6, 128.0), turned to 180 degrees
- moved R13 140.8 mm to (140.4, 138.3), turned to -90 degrees
- moved J2 138.2 mm to (144.0, 138.7), turned to 180 degrees
- moved C17 137.6 mm to (154.2, 116.5)
- moved C18 129.4 mm to (135.1, 129.9), turned to 180 degrees
- moved R4 129.4 mm to (142.7, 115.8)
- moved SW1 128.4 mm to (124.2, 138.8), turned to 90 degrees
- moved SW2 128.0 mm to (137.3, 132.2), turned to -90 degrees
- moved R8 127.5 mm to (148.7, 115.0), turned to 180 degrees
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Routing:
- net +3.3V: track 0.00 -> 229.8 mm
- net GND: track 0.00 -> 58.4 mm, vias 0 -> 25
- net +5V: track 0.00 -> 55.6 mm, vias 0 -> 5
- net USB_DM: track 0.00 -> 43.5 mm
- net USB_DP: track 0.00 -> 40.4 mm
- net VBUS: track 0.00 -> 10.2 mm
- net Net-(D1-A): track 0.00 -> 7.06 mm
- added copper zone on F.Cu, net +3.3V
- added copper zone on B.Cu, net GND

Commit message: after resizing
Parts:
- moved J4 48.0 mm to (123.3, 155.3)
- moved J5 38.0 mm to (122.7, 107.3)
- moved R13 37.4 mm to (173.8, 155.1)
- moved SW1 36.0 mm to (155.9, 155.7)
- moved SW2 36.0 mm to (169.1, 149.2)
- moved R3 26.3 mm to (173.9, 134.6)
- moved J2 25.6 mm to (169.2, 134.0)
- moved H4 18.0 mm to (181.0, 156.0)
- moved C15 15.0 mm to (180.2, 140.0)
- moved C16 15.0 mm to (176.6, 136.8)
- moved H2 15.0 mm to (181.0, 104.0)
- moved Q1 15.0 mm to (181.5, 128.6)
- moved R5 15.0 mm to (182.1, 132.9)
- moved R6 15.0 mm to (178.4, 134.2)
- moved R7 15.0 mm to (176.6, 128.0)
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Connections:
- J5 pad 10: PA4 -> PA7
- J5 pad 11: PB0 -> PA6
- J5 pad 12: PB1 -> PA4
- J5 pad 13: PA6 -> PA1
- J5 pad 14: PA7 -> PC3
- J5 pad 15: PA8 -> PC2
- J5 pad 16: PA15 -> PC1
- J5 pad 17: PB6 -> PC0
- J5 pad 18: PB7 -> PB6
- J5 pad 19: PC9 -> PB7
- J5 pad 3: PC0 -> PA15
- J5 pad 4: PC1 -> PA8
- J5 pad 5: PC2 -> PC9
- J5 pad 6: PC3 -> PB1
- J5 pad 7: PC4 -> PB0
- J5 pad 9: PA1 -> PC4
Routing:
- net +3.3V: track 229.8 -> 289.7 mm, vias 0 -> 3
- net SWO: track 0.00 -> 53.3 mm, vias 0 -> 1
- net SWDIO: track 0.00 -> 49.4 mm, vias 0 -> 1
- net PB6: track 0.00 -> 43.1 mm, vias 0 -> 4
- net PC2: track 0.00 -> 42.1 mm, vias 0 -> 4
- net PC1: track 0.00 -> 39.9 mm, vias 0 -> 2
- net GND: track 58.4 -> 97.8 mm, vias 25 -> 29
- net SWCLK: track 0.00 -> 38.4 mm, vias 0 -> 1
- net LED_STATUS: track 0.00 -> 38.1 mm, vias 0 -> 2
- net PA8: track 0.00 -> 34.0 mm, vias 0 -> 5
- net NRST: track 0.00 -> 32.4 mm, vias 0 -> 3
- net PC3: track 0.00 -> 32.4 mm, vias 0 -> 2
- net LED_USER_1: track 0.00 -> 29.3 mm
- net PA15: track 0.00 -> 29.3 mm, vias 0 -> 4
- net PA1: track 0.00 -> 28.6 mm, vias 0 -> 5
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Other:
- board size 70 x 50 mm -> 85 x 60 mm

Commit message: Remaped headers, routed the mcu and j4,j5, almost finished
Parts:
- moved J3 55.7 mm to (121.0, 141.7), turned to 90 degrees
- moved J5 6.14 mm to (128.1, 104.4)
- moved J4 3.58 mm to (125.9, 157.7)
- moved C10 0.24 mm to (150.8, 117.3)
- moved U4 0.10 mm to (182.6, 136.9)
- turned C6 to 90 degrees
Connections:
- net I2C2_SDA renamed PC12
- J4 pad 10: I2C1_SDA -> PC10
- J4 pad 11: I2C2_SCL -> PC11
- J4 pad 13: SPI2_NSS -> PD2
- J4 pad 14: SPI2_SCK -> USART1_TX
- J4 pad 15: SPI2_MISO -> USART1_RX
- J4 pad 16: SPI2_MOSI -> I2C1_SCL
- J4 pad 17: PC10 -> I2C1_SDA
- J4 pad 18: PC11 -> PC0
- J4 pad 19: PD2 -> PC1
- J4 pad 5: USART2_TX -> PC9
- J4 pad 6: USART2_RX -> PA8
- J4 pad 7: USART1_TX -> PA9
- J4 pad 8: USART1_RX -> PA10
- J4 pad 9: I2C1_SCL -> PA15
- J5 pad 10: PA7 -> PC5
- J5 pad 11: PA6 -> PC4
- J5 pad 12: PA4 -> PA7
- J5 pad 13: PA1 -> PA6
- J5 pad 14: PC3 -> PA4
- J5 pad 15: PC2 -> USART2_RX
- J5 pad 16: PC1 -> USART2_TX
- J5 pad 17: PC0 -> PA1
- J5 pad 18: PB6 -> PC3
- J5 pad 19: PB7 -> PC2
- J5 pad 3: PA15 -> SPI2_MOSI
- J5 pad 4: PA8 -> SPI2_MISO
- J5 pad 5: PC9 -> SPI2_SCK
- J5 pad 6: PB1 -> SPI2_NSS
- J5 pad 7: PB0 -> PB10
- J5 pad 8: PC5 -> PB1
- J5 pad 9: PC4 -> PB0
- U3 pad 29: I2C2_SCL -> PB10
- U3 pad 42: USART1_TX -> PA9
- U3 pad 43: USART1_RX -> PA10
- U3 pad 58: PB6 -> USART1_TX
- U3 pad 59: PB7 -> USART1_RX
Routing:
- net I2C1_SCL: track 4.23 -> 87.6 mm, vias 0 -> 1
- net I2C1_SDA: track 7.41 -> 79.4 mm, vias 2 -> 3
- net Net-(Q1-Pad1): track 2.34 -> 68.3 mm, vias 0 -> 4
- net BTN_USER: track 4.79 -> 58.9 mm, vias 0 -> 2
- net PA9: track 0.00 -> 47.3 mm, vias 0 -> 1
- net PB6: track 43.1 -> 0.00 mm, vias 4 -> 0
- net NRST: track 32.4 -> 74.5 mm, vias 3 -> 1
- net PA10: track 0.00 -> 40.7 mm, vias 0 -> 1
- net SWO: track 53.3 -> 15.7 mm
- net PC10: track 0.00 -> 36.3 mm, vias 0 -> 1
- net PC11: track 0.00 -> 33.8 mm, vias 0 -> 1
- net Net-(J2-Pin_1): track 4.13 -> 34.0 mm, vias 0 -> 1
- net PD2: track 0.00 -> 29.6 mm, vias 0 -> 1
- net USART1_TX: track 0.00 -> 29.3 mm, vias 0 -> 1
- net USART1_RX: track 0.00 -> 29.2 mm, vias 0 -> 1
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
Commit message: silkscreen left to do
Parts:
- moved C18 41.9 mm to (172.3, 149.2), turned to 0 degrees
Routing:
- net I2C1_SDA: track 79.4 -> 104.8 mm
- net PD2: track 29.6 -> 49.4 mm
- net PC12: track 26.5 -> 45.3 mm
- net SPI2_MISO: track 28.3 -> 46.8 mm
- net +3.3V: track 292.8 -> 304.7 mm
- net BTN_USER: track 58.9 -> 47.2 mm
- net PC11: track 33.8 -> 43.2 mm
- net SPI2_SCK: track 21.9 -> 31.2 mm
- net SPI2_NSS: track 20.8 -> 28.4 mm
- net SWO: track 15.7 -> 22.1 mm
- net PA15: track 34.5 -> 40.2 mm
- net NRST: track 74.5 -> 80.0 mm
- net PC10: track 36.3 -> 40.9 mm
- net SPI2_MOSI: track 27.8 -> 31.7 mm
- net GND: track 110.4 -> 106.6 mm, vias 29 -> 95
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- added copper zone on F.Cu, net GND

Commit message: final version of pcb, configured silkscreen, text and ready to generate gerber files
Routing:
- net GND: track 106.6 -> 123.1 mm, vias 95 -> 96
Other:
- board text added: "ANALOG/GPIO"
- board text added: "BOOT0"
- board text added: "COMM"
- board text added: "M. Haftarczyk 2026"
- board text added: "PWR"
- board text added: "RESET"
- board text added: "STAT"
- board text added: "STM32F446 DEV BOARD"
- board text added: "SWD"
- board text added: "USB 5V"
- board text added: "USER"
- board text added: "USR1"
- board text added: "USR2"
- board text added: "USR3"
